File: ethernet.kicad_sch (KiCad schematic)
At the start: 9 parts, among them J1 HR911105A

Commit message: Updated BOM
Parts:
- C48, C49: LCSC Part # (none) -> C131394
- C51, C52, C56, C57: LCSC Part # (none) -> C60133
- J1: LCSC Part Num (none) -> C12074
- R13, R14: LCSC Part # (none) -> C25104
