File: SBC.kicad_pcb (KiCad board)
At the start: 4 copper layers, 100 x 60.1 mm, 146 parts, among them J1 HR911105A, J2 Conn_01x07_Socket, J3 Wire_Solder_2Pin, Q4 DOD40P03, U1 Allwinner_V3s, U2 TPS54331DR, U3 TPS54331DR, U4 TPS54331DR, U5 TLV1117-33, U6 TLV1117-18, U7 RP2040, U8 W25Q16JVSS, Y1 Crystal_GND24, Y2 Crystal_GND24

Commit message: Rev1
Connections:
- U1 pad 85: unconnected-(U1B-VCC-MCSI-Pad85) -> +3.3V
Routing:
- net +3.3V: track 205.4 -> 211.4 mm
- net Net-(U7-~{QSPI_SS}): track 15.4 -> 16.5 mm
- net GND: vias 275 -> 518
Other:
- board text added: "Allwinner V3S Rev 1 Sept 21 2026 Michael Yablonovitch"

Commit message: updayted BOM, fixed inductor values
Parts:
- C46, C47: value 36p -> 18p
- Y1: value Crystal_GND24 -> 24 MHz
- Y2: value Crystal_GND24 -> 12 MHz
Changed lines of the file:
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@@
 			)
 		)
-		(attr smd dnp)
+		(attr smd)
 		(duplicate_pad_numbers_are_jumpers no)
 		(fp_line
@@
 			)
 		)
-		(attr smd dnp)
+		(attr smd)
 		(duplicate_pad_numbers_are_jumpers no)
 		(fp_line
@@
 			)
 		)
-		(property "LCSC Part #" "C14664"
+		(property "LCSC Part #" "C596327"
 			(at 0 0 180)
 			(unlocked yes)
@@
 			)
 		)
-		(property "Value" "36p"
+		(property "Value" "18p"
 			(at 0 1.43 0)
 			(layer "F.Fab")
@@
 			)
 		)
-		(property "LCSC Part #" "C519462"
+		(property "LCSC Part #" "C107040"
 			(at 0 0 180)
 			(unlocked yes)
@@
 			)
 		)
-		(property "LCSC Part #" "C14664"
+		(property "LCSC Part #" "C596327"
 			(at 0 0 270)
 			(unlocked yes)
@@
 			)
 		)
-		(attr smd dnp)
+		(attr smd)
 		(duplicate_pad_numbers_are_jumpers no)
 		(fp_line
@@
 			)
 		)
-		(attr smd dnp)
+		(attr smd)
 		(duplicate_pad_numbers_are_jumpers no)
 		(fp_line
@@
 			)
 		)
-		(attr smd dnp)
+		(attr smd)
 		(duplicate_pad_numbers_are_jumpers no)
 		(fp_line
@@
 			)
 		)
-		(property "Value" "Crystal_GND24"
+		(property "Value" "12 MHz"
 			(at 0 2.45 90)
 			(layer "F.Fab")
@@
 			)
 		)
-		(property "LCSC Part #" "C13738"
+		(property "LCSC Part #" "C50430"
 			(at 0 0 270)
 			(unlocked yes)
@@
 			)
 		)
-		(property "LCSC Part #" "C167220"
+		(property "LCSC Part #" "C167219"
 			(at 0 0 270)
 			(unlocked yes)
@@
 			)
 		)
-		(attr smd dnp)
+		(attr smd)
 		(duplicate_pad_numbers_are_jumpers no)
 		(fp_line
@@
 			)
 		)
-		(property "Value" "Crystal_GND24"
+		(property "Value" "24 MHz"
 			(at 0 2.45 270)
 			(layer "F.Fab")
@@
 			)
 		)
-		(property "LCSC Part #" "C12260"
+		(property "LCSC Part #" "C70590"
 			(at 0 0 270)
 			(unlocked yes)
@@
 			)
 		)
-		(property "Value" "36p"
+		(property "Value" "18p"
 			(at 0 1.43 0)
 			(layer "F.Fab")
@@
 			)
 		)
-		(property "LCSC Part #" "C519462"
+		(property "LCSC Part #" "C107040"
 			(at 0 0 0)
 			(unlocked yes)
@@
 			)
 		)
-		(property "LCSC Part #" "C167222"
+		(property "LCSC Part #" "C167221"
 			(at 0 0 270)
 			(unlocked yes)
