File: SBC.kicad_sch (KiCad schematic)
At the start: 23 parts, among them U1 Allwinner_V3s, Y1 Crystal_GND24

Commit message: did some routing
Parts:
- added C67: 4u7, Capacitor_SMD:C_0603_1608Metric_Pad1.08x0.95mm_HandSolder, symbol Device:C
- Y1: footprint Crystal:Crystal_SMD_3225-4Pin_3.2x2.5mm_HandSoldering -> Crystal:Crystal_SMD_3225-4Pin_3.2x2.5mm
Connections:
- net +1V8: now also C67.2
- net GND: now also U1.EPAD (EGND), C67.1; no longer U1.129 (EGND)
Changed lines of the file:
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@@
 	)
 	(junction
-		(at 143.51 152.4)
-		(diameter 0)
-		(color 0 0 0 0)
-	)
-	(junction
 		(at 100.33 77.47)
 		(diameter 0)
@@
 	)
 	(junction
+		(at 273.05 116.84)
+		(diameter 0)
+		(color 0 0 0 0)
+	)
+	(junction
 		(at 100.33 113.03)
 		(diameter 0)
@@
 	)
 	(junction
+		(at 143.51 152.4)
+		(diameter 0)
+		(color 0 0 0 0)
+	)
+	(junction
 		(at 220.98 116.84)
 		(diameter 0)
@@
 	(wire
 		(pts
-			(xy 269.24 99.06) (xy 269.24 116.84)
+			(xy 273.05 99.06) (xy 273.05 116.84)
 		)
 		(stroke
@@
 	(wire
 		(pts
-			(xy 260.35 116.84) (xy 269.24 116.84)
+			(xy 260.35 116.84) (xy 273.05 116.84)
 		)
 		(stroke
@@
 		(pin "97"
 		)
-		(pin "129"
+		(pin "EPAD"
 		)
 		(pin "98"
@@
 	)
 	(symbol
+		(lib_id "Device:C")
+		(at 273.05 120.65 180)
+		(unit 1)
+		(body_style 1)
+		(exclude_from_sim no)
+		(in_bom yes)
+		(on_board yes)
+		(in_pos_files yes)
+		(dnp no)
+		(fields_autoplaced yes)
+		(property "Reference" "C67"
+			(at 276.86 119.3799 0)
+			(show_name no)
+			(do_not_autoplace no)
+			(effects
+				(font
+					(size 1.27 1.27)
+				)
+				(justify right)
+			)
+		)
+		(property "Value" "4u7"
+			(at 276.86 121.9199 0)
+			(show_name no)
+			(do_not_autoplace no)
+			(effects
+				(font
+					(size 1.27 1.27)
+				)
+				(justify right)
+			)
+		)
+		(property "Footprint" "Capacitor_SMD:C_0603_1608Metric_Pad1.08x0.95mm_HandSolder"
+			(at 272.0848 116.84 0)
+			(hide yes)
+			(show_name no)
+			(do_not_autoplace no)
+			(effects
+				(font
+					(size 1.27 1.27)
+				)
+			)
+		)
+		(property "Datasheet" ""
+			(at 273.05 120.65 0)
+			(hide yes)
+			(show_name no)
+			(do_not_autoplace no)
+			(effects
+				(font
+					(size 1.27 1.27)
+				)
+			)
+		)
+		(property "Description" "Unpolarized capacitor"
+			(at 273.05 120.65 0)
+			(hide yes)
+			(show_name no)
+			(do_not_autoplace no)
+			(effects
+				(font
+					(size 1.27 1.27)
+				)
+			)
+		)
+		(pin "1"
+		)
+		(pin "2"
+		)
+		(instances
+			(project "SBC"
+				(path "/b4d218fa-7dac-4029-a1de-f18f86a4abe3"
+					(reference "C67")
+					(unit 1)
+				)
+			)
+		)
+	)
+	(symbol
 		(lib_id "power:GND")
 		(at 207.01 60.96 0)
@@
 	(symbol
 		(lib_id "power:+1V8")
-		(at 269.24 99.06 0)
+		(at 273.05 99.06 0)
 		(unit 1)
 		(body_style 1)
@@
 		(fields_autoplaced yes)
 		(property "Reference" "#PWR035"
-			(at 269.24 102.87 0)
+			(at 273.05 102.87 0)
 			(hide yes)
 			(show_name no)
@@
 		)
 		(property "Value" "+1V8"
-			(at 269.24 93.98 0)
+			(at 273.05 93.98 0)
 			(show_name no)
 			(do_not_autoplace no)
@@
 		)
 		(property "Footprint" ""
-			(at 269.24 99.06 0)
+			(at 273.05 99.06 0)
 			(hide yes)
 			(show_name no)
@@
 		)
 		(property "Datasheet" ""
-			(at 269.24 99.06 0)
+			(at 273.05 99.06 0)
 			(hide yes)
 			(show_name no)
@@
 		)
 		(property "Description" "Power symbol creates a global label with name \"+1V8\""
-			(at 269.24 99.06 0)
+			(at 273.05 99.06 0)
 			(hide yes)
 			(show_name no)
@@
 	)
 	(symbol
+		(lib_id "power:GND")
+		(at 273.05 124.46 0)
+		(unit 1)
+		(body_style 1)
+		(exclude_from_sim no)
+		(in_bom yes)
+		(on_board yes)
+		(in_pos_files yes)
+		(dnp no)
+		(fields_autoplaced yes)
+		(property "Reference" "#PWR098"
+			(at 273.05 130.81 0)
+			(hide yes)
+			(show_name no)
+			(do_not_autoplace no)
+			(effects
+				(font
+					(size 1.27 1.27)
+				)
+			)
+		)
+		(property "Value" "GND"
+			(at 273.05 129.54 0)
+			(show_name no)
+			(do_not_autoplace no)
+			(effects
+				(font
+					(size 1.27 1.27)
+				)
+			)
+		)
+		(property "Footprint" ""
+			(at 273.05 124.46 0)
+			(hide yes)
+			(show_name no)
+			(do_not_autoplace no)
+			(effects
+				(font
+					(size 1.27 1.27)
+				)
+			)
+		)
+		(property "Datasheet" ""
+			(at 273.05 124.46 0)
+			(hide yes)
+			(show_name no)
+			(do_not_autoplace no)
+			(effects
+				(font
+					(size 1.27 1.27)
+				)
+			)
+		)
+		(property "Description" "Power symbol creates a global label with name \"GND\" , ground"
+			(at 273.05 124.46 0)
+			(hide yes)
+			(show_name no)
+			(do_not_autoplace no)
+			(effects
+				(font
+					(size 1.27 1.27)
+				)
+			)
+		)
+		(pin "1"
+		)
+		(instances
+			(project "SBC"
+				(path "/b4d218fa-7dac-4029-a1de-f18f86a4abe3"
+					(reference "#PWR098")
+					(unit 1)
+				)
+			)
+		)
+	)
+	(symbol
 		(lib_id "Device:C")
 		(at 60.96 119.38 180)
@@
 			)
 		)
-		(property "Footprint" "Crystal:Crystal_SMD_3225-4Pin_3.2x2.5mm_HandSoldering"
+		(property "Footprint" "Crystal:Crystal_SMD_3225-4Pin_3.2x2.5mm"
 			(at 207.01 50.8 0)
 			(hide yes)

Commit message: Rev1
Connections:
- net +3.3V: now also U1.85 (VCC-MCSI)
Changed lines of the file:
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@@
+	)
+	(junction
+		(at 100.33 87.63)
+		(diameter 0)
+		(color 0 0 0 0)
 	)
 	(junction
@@
 	(wire
 		(pts
+			(xy 100.33 87.63) (xy 116.84 87.63)
+		)
+		(stroke
+			(width 0)
+			(type default)
+		)
+	)
+	(wire
+		(pts
 			(xy 187.96 67.31) (xy 187.96 50.8)
 		)
@@
 	(wire
 		(pts
-			(xy 100.33 92.71) (xy 100.33 77.47)
+			(xy 100.33 92.71) (xy 100.33 87.63)
 		)
 		(stroke
@@
 		)
 		(stroke
+			(width 0)
+			(type default)
+		)
+	)
+	(wire
+		(pts
+			(xy 100.33 87.63) (xy 100.33 77.47)
+		)
+		(stroke

Commit message: Updated BOM
Parts:
- C31: LCSC Part # (none) -> C14664
- C32, C33, C34, C35, C36, C37, C40, C41, C42, C43, C44, C45: LCSC Part # (none) -> C1591
- C38, C39, C67: LCSC Part # (none) -> C296042
- C46, C47: LCSC Part # (none) -> C519462
- FB1: LCSC Part # (none) -> C341663
- R10: LCSC Part # (none) -> C22772
- R11: LCSC Part # (none) -> C23350
- R12: LCSC Part # (none) -> C25804
- Y1: LCSC Part Num (none) -> C12260

Commit message: updayted BOM, fixed inductor values
Parts:
- C46, C47: value 36p -> 18p; LCSC Part # C519462 -> C107040
- Y1: value Crystal_GND24 -> 24 MHz; LCSC Part # C12260 -> C70590
Changed lines of the file:
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@@
 			)
 		)
-		(property "Value" "36p"
+		(property "Value" "18p"
 			(at 199.39 58.4199 0)
 			(show_name no)
@@
 			)
 		)
-		(property "LCSC Part #" "C519462"
+		(property "LCSC Part #" "C107040"
 			(at 195.58 57.15 0)
 			(hide yes)
@@
 			)
 		)
-		(property "Value" "36p"
+		(property "Value" "18p"
 			(at 219.71 58.4199 0)
 			(show_name no)
@@
 			)
 		)
-		(property "LCSC Part #" "C519462"
+		(property "LCSC Part #" "C107040"
 			(at 215.9 57.15 0)
 			(hide yes)
@@
 			)
 		)
-		(property "Value" "Crystal_GND24"
+		(property "Value" "24 MHz"
 			(at 207.01 44.45 0)
 			(show_name no)
@@
 			)
 		)
-		(property "LCSC Part #" "C12260"
+		(property "LCSC Part #" "C70590"
 			(at 207.01 50.8 0)
 			(hide yes)
