File: cmsis_dap_programmer.kicad_sch (KiCad schematic)
At the start: 39 parts, among them J2 Conn_01x07_Socket, U7 RP2040, U8 W25Q16JVSS, Y2 Crystal_GND24

Commit message: Updated BOM
Parts:
- C53, C59, C66, C68, C71: LCSC Part # (none) -> C14664
- C54, C58, C60, C61, C65, C69, C70, C72, C74: LCSC Part # (none) -> C1591
- C63, C64: LCSC Part # (none) -> C107037
- D13, D4, D6: LCSC Part # (none) -> C8657
- D15, D16, D18, D19, D20: LCSC Part # (none) -> C3040608
- J2: LCSC Part # (none) -> C17565513
- R22, R32: LCSC Part # (none) -> C25099
- R30, R31: LCSC Part Num (none) -> C98220
- R33: LCSC Part # (none) -> C25077
- R34, R35, R36, R37, R38, R39: LCSC Part # (none) -> C25076
- U7: LCSC Part # (none) -> C2040
- U8: LCSC Part Num (none) -> C131025
- Y2: LCSC Part Num (none) -> C13738

Commit message: updayted BOM, fixed inductor values
Parts:
- Y2: value Crystal_GND24 -> 12 MHz; LCSC Part # C13738 -> C50430
Changed lines of the file:
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@@
 			)
 		)
-		(property "Value" "Crystal_GND24"
+		(property "Value" "12 MHz"
 			(at 97.79 127 0)
 			(show_name no)
@@
 			)
 		)
-		(property "LCSC Part #" "C13738"
+		(property "LCSC Part #" "C50430"
 			(at 97.79 133.35 0)
 			(hide yes)
