File: power.kicad_sch (KiCad schematic)
At the start: 50 parts, among them U2 TPS54331DR, U3 TPS54331DR, U4 TPS54331DR, U5 TLV1117-33, U6 TLV1117-18

Commit message: did some routing
Parts:
- added C50: 100u, Capacitor_THT:CP_Radial_D8.0mm_P3.50mm, symbol Device:C_Polarized
- added D10, D11, D12, D7, D8, D9: LED, LED_SMD:LED_0805_2012Metric_Pad1.15x1.40mm_HandSolder, symbol Device:LED
- added D5: BZT52C10, Diode_SMD:D_SOD-123F, symbol Diode:BZT52Bxx
- added F2: Fuse, Fuse:Fuseholder_Clip-5x20mm_Bel_FC-203-22_Lateral_P17.80x5.00mm_D1.17mm_Horizontal, symbol Device:Fuse
- added J3: Wire_Solder_2Pin, HighCurrent_Wire_Solder:Wire_Solder_2Pin_12-14AWG_P10mm_D3.0mm, symbol HighCurrent_Wire_Solder:Wire_Solder_2Pin
- added Q4: DOD40P03, DOINGTER:DOD40P03_TO-252_Q_PMOS_DGS, symbol Transistor_FET:Q_PMOS_DGS
- added R17, R18, R19, R20, R21: 0r, Resistor_SMD:R_0603_1608Metric, symbol Device:R
- added R23, R24, R25, R26, R27, R28, R29: 10k, Resistor_SMD:R_0603_1608Metric_Pad0.98x0.95mm_HandSolder, symbol Device:R
- R2, R6, R9: footprint (none) -> Resistor_SMD:R_0603_1608Metric
Connections:
- net +12V: now also C50.1, D5.1 (K), D7.2 (A), Q4.3 (S)
- net +1V2: now also R20.2; no longer C23.1, C24.1, L3.2, R8.1
- net +1V8: now also R19.2; no longer C29.2, C30.2, U6.2 (VO)
- net +3.3V: now also R18.2; no longer C15.1, C16.1, L2.2, R5.1
- net +3.3VA: now also R21.2; no longer C26.2, C27.2, U5.2 (VO)
- net +5V: now also R17.2; no longer C7.1, C8.1, L1.2, R1.1
- net GND: now also C50.2, J3.1 (WIRE1), R23.1, R24.1, R25.1, R26.1, R27.1, R28.1, R29.1
- new net: C7.1, C8.1, D11.2 (A), L1.2, R1.1, R17.1
- new net: D10.1 (K), R27.2
- new net: C23.1, C24.1, D10.2 (A), L3.2, R20.1, R8.1
- new net: C26.2, C27.2, D12.2 (A), R21.1, U5.2 (VO)
- new net: D7.1 (K), R24.2
- new net: C15.1, C16.1, D8.2 (A), L2.2, R18.1, R5.1
- new net: C29.2, C30.2, D9.2 (A), R19.1, U6.2 (VO)
- new net: D8.1 (K), R25.2
- new net: D12.1 (K), R29.2
- new net: D5.2 (A), Q4.2 (G), R23.2
- new net: F2.1, J3.2 (WIRE2)
- new net: D9.1 (K), R26.2
- new net: D11.1 (K), R28.2
- new net: F2.2, Q4.1 (D)
Other:
- moved on the sheet: C1, C10, C11, C12, C13, C14, C15, C16, C17, C18, C19, C2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

Commit message: Updated BOM
Parts:
- C1, C17, C21, C9: LCSC Part # (none) -> C100042
- C10, C18, C5: LCSC Part # (none) -> C2909422
- C11, C6: LCSC Part # (none) -> C105622
- C12, C14, C2, C20, C22, C3: LCSC Part # (none) -> C1591
- C13: LCSC Part # (none) -> C106218
- C15, C16, C23, C24, C7, C8: LCSC Part # (none) -> C596320
- C19: LCSC Part # (none) -> C14665
- C25, C26, C27, C28, C29, C30: LCSC Part # (none) -> C14664
- C4: LCSC Part # (none) -> C107088
- C50: LCSC Part Num (none) -> C171434
- D1, D2, D3: LCSC Part # (none) -> C3759261
- D10, D11, D12, D7, D8, D9: LCSC Part Num (none) -> C110099; now not fitted
- D5: LCSC Part Num (none) -> C571378
- F2: LCSC Part # (none) -> C3205463
- L1: LCSC Part Num (none) -> C167223
- L2: LCSC Part Num (none) -> C167222
- L3: LCSC Part Num (none) -> C167220
- Q4: LCSC Part Num (none) -> C36499177
- R1, R3, R5, R8: LCSC Part # (none) -> C22772
- R17, R18, R19, R20, R21: LCSC Part # (none) -> C21189
- R2: LCSC Part # (none) -> C22850
- R23, R24, R25, R26, R27, R28, R29: LCSC Part Num (none) -> C98220
- R4: LCSC Part # (none) -> C23212
- R6: LCSC Part # (none) -> C22994
- R7: LCSC Part # (none) -> C22978
- R9: LCSC Part # (none) -> C22910
- U2, U3, U4: LCSC Part # (none) -> C9865
- U5: LCSC Part # (none) -> C37359
- U6: LCSC Part # (none) -> C2862410

Commit message: updayted BOM, fixed inductor values
Parts:
- C26, C30: LCSC Part # C14664 -> C596327
- D10, D11, D12, D7, D8, D9: now fitted
- L2: LCSC Part # C167222 -> C167221
- L3: LCSC Part # C167220 -> C167219
Changed lines of the file:
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@@
 		(on_board yes)
 		(in_pos_files yes)
-		(dnp yes)
+		(dnp no)
 		(fields_autoplaced yes)
 		(property "Reference" "D10"
@@
 		(on_board yes)
 		(in_pos_files yes)
-		(dnp yes)
+		(dnp no)
 		(fields_autoplaced yes)
 		(property "Reference" "D7"
@@
 			)
 		)
-		(property "LCSC Part #" "C167222"
+		(property "LCSC Part #" "C167221"
 			(at 162.56 186.69 90)
 			(hide yes)
@@
 		(on_board yes)
 		(in_pos_files yes)
-		(dnp yes)
+		(dnp no)
 		(fields_autoplaced yes)
 		(property "Reference" "D11"
@@
 		(on_board yes)
 		(in_pos_files yes)
-		(dnp yes)
+		(dnp no)
 		(fields_autoplaced yes)
 		(property "Reference" "D8"
@@
 			)
 		)
-		(property "LCSC Part #" "C14664"
+		(property "LCSC Part #" "C596327"
 			(at 514.35 78.74 0)
 			(hide yes)
@@
 		(on_board yes)
 		(in_pos_files yes)
-		(dnp yes)
+		(dnp no)
 		(fields_autoplaced yes)
 		(property "Reference" "D9"
@@
 		(on_board yes)
 		(in_pos_files yes)
-		(dnp yes)
+		(dnp no)
 		(fields_autoplaced yes)
 		(property "Reference" "D12"
@@
 			)
 		)
-		(property "LCSC Part #" "C14664"
+		(property "LCSC Part #" "C596327"
 			(at 269.24 194.31 0)
 			(hide yes)
@@
 			)
 		)
-		(property "LCSC Part #" "C167220"
+		(property "LCSC Part #" "C167219"
 			(at 441.96 184.15 90)
 			(hide yes)
